File: custom_keypad/custom_keypad.sch (KiCad schematic (older format))
At the start: 1 part

Commit message: Schematic design
Parts:
- added C1, C4, C6: 0.1uF, Capacitor_SMD:C_0805_2012Metric, symbol Device:C_Small
- added C2, C3: 22pF, Capacitor_SMD:C_0805_2012Metric, symbol Device:C_Small
- added C5: 1uF, Capacitor_SMD:C_0805_2012Metric, symbol Device:C_Small
- added C7: 10uF, Capacitor_SMD:C_0805_2012Metric, symbol Device:C_Small
- added D1, D2, D3, D4: D_Small, Diode_SMD:D_SOD-123, symbol Device:D_Small
- added F1: 500mA, Fuse:Fuse_1206_3216Metric, symbol Device:Polyfuse_Small
- added MX1, MX2, MX3, MX4: MX-NoLED, MX_Alps_Hybrid:MX-1U, symbol MX_Alps_Hybrid:MX-NoLED
- added R1, R2: 22, Resistor_SMD:R_0805_2012Metric, symbol Device:R_Small
- added R3, R4: 10k, Resistor_SMD:R_0805_2012Metric, symbol Device:R_Small
- added SW1: SW_Push, random-keyboard-parts:SKQG-1155865, symbol Switch:SW_Push
- added USB1: Molex-0548190589, random-keyboard-parts:Molex-0548190589, symbol random-keyboard-parts:Molex-0548190589
- added Y1: 16MHz, Crystal:Crystal_SMD_3225-4Pin_3.2x2.5mm, symbol Device:Crystal_GND24_Small
- gave numbers to parts that had none: 1
Connections:
- net +5V: now also U1.7 (VBUS), C1.1, C4.1, C6.1, C7.1, F1.1, R3.1
- net at U1.13 (~RESET): now also R3.2, SW1.2
- net GND: now reaches U1.15 (GND), U1.23 (GND), U1.35 (GND), U1.43 (GND)
- net GND: now also U1.5 (UGND), C1.2, C2.2, C3.2, C4.2, C5.2, C6.2, C7.2, R4.1, SW1.1, USB1.1 (GND), Y1.2, Y1.4
- net at U1.16 (XTAL2): now also C3.1, Y1.3
- net at U1.17 (XTAL1): now also C2.1, Y1.1
- net at U1.3 (D-): now also R1.1
- net at U1.33 (~HWB~/PE2): now also R4.2
- net at U1.4 (D+): now also R2.1
- net at U1.6 (UCAP): now also C5.1
- new net: D1.2 (A), MX1.2 (ROW)
- new net: D3.2 (A), MX3.2 (ROW)
- new net: D2.2 (A), MX2.2 (ROW)
- new net: D4.2 (A), MX4.2 (ROW)
- new net COL0: MX1.1 (COL), MX2.1 (COL)
- new net COL1: MX3.1 (COL), MX4.1 (COL)
- new net D+: R2.2, USB1.3 (D+)
- new net D-: R1.2, USB1.4 (D-)
- new net ROW0: D1.1 (K), D3.1 (K)
- new net ROW1: D2.1 (K), D4.1 (K)
- new net VCC: F1.2, USB1.5 (VBUS)
Other:
- moved on the sheet: U1
